File: PCB/Catie Hackpad.kicad_pcb (KiCad board)
At the start: 2 copper layers, 20.6 x 100.1 mm, 9 parts, among them SW1 SW_Push, SW2 SW_Push, SW3 SW_Push, SW4 SW_Push, U1 XIAO-RP2040-DIP

Commit message: Add files via upload
Parts:
- D1, D2, D3, D4: value SK6812 -> LED_SK6812MINI; footprint LED_SMD:LED_SK6812MINI_PLCC4_3.5x3.5mm_P1.75mm -> Hackclub Footprints:MX_SK6812MINI-E_REV
- U1: footprint Seeed Studio XIAO Series Library:XIAO-RP2040-DIP -> Hackclub Footprints:XIAO-RP2040-DIP
- moved D3 9.53 mm to (114.3, 95.2)
- moved D4 9.53 mm to (114.3, 114.3)
- moved D1 9.52 mm to (114.3, 57.1)
- moved D2 9.52 mm to (114.3, 76.2)
Connections:
- D1 pad 1: GND -> +5V
- D1 pad 2: Net-(D1-DIN) -> Net-(D1-DOUT)
- D1 pad 3: +5V -> GND
- D1 pad 4: Net-(D1-DOUT) -> Net-(D1-DIN)
- D2 pad 1: GND -> +5V
- D2 pad 2: Net-(D1-DOUT) -> Net-(D2-DOUT)
- D2 pad 3: +5V -> GND
- D2 pad 4: Net-(D2-DOUT) -> Net-(D1-DOUT)
- D3 pad 1: GND -> +5V
- D3 pad 2: Net-(D2-DOUT) -> Net-(D3-DOUT)
- D3 pad 3: +5V -> GND
- D3 pad 4: Net-(D3-DOUT) -> Net-(D2-DOUT)
- D4 pad 1: GND -> +5V
- D4 pad 2: Net-(D3-DOUT) -> unconnected-(D4-DOUT-Pad2)
- D4 pad 3: +5V -> GND
- D4 pad 4: Net-(D4-DOUT) -> Net-(D3-DOUT)
Routing:
- net GND: track 116.2 -> 127.6 mm, vias 0 -> 1
- net +5V: track 118.4 -> 108.1 mm, vias 0 -> 4
- net Net-(D1-DIN): track 39.1 -> 31.6 mm, vias 3 -> 0
- net Net-(D2-DOUT): track 28.7 -> 26.4 mm, vias 2 -> 0
- net Net-(D1-DOUT): track 28.7 -> 26.4 mm, vias 2 -> 0
- net Net-(D3-DOUT): track 27.7 -> 26.4 mm
Other:
- board size 20.6 x 100.1 mm -> 20.6 x 100 mm
