File: PCB/Catie Hackpad.kicad_sch (KiCad schematic)
At the start: 9 parts, among them SW1 SW_Push, SW2 SW_Push, SW3 SW_Push, SW4 SW_Push, U1 XIAO-RP2040-DIP

Commit message: Add files via upload
Parts:
- D1, D2, D3, D4: footprint ScottoKeebs_Components:LED_SK6812MINI -> Hackclub Footprints:MX_SK6812MINI-E_REV
- U1: footprint Seeed Studio XIAO Series Library:XIAO-RP2040-DIP -> Hackclub Footprints:XIAO-RP2040-DIP
Changed lines of the file:
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@@
 			)
 		)
-		(property "Footprint" "ScottoKeebs_Components:LED_SK6812MINI"
+		(property "Footprint" "Hackclub Footprints:MX_SK6812MINI-E_REV"
 			(at 109.22 59.69 0)
 			(effects
@@
 			)
 		)
-		(property "Footprint" "ScottoKeebs_Components:LED_SK6812MINI"
+		(property "Footprint" "Hackclub Footprints:MX_SK6812MINI-E_REV"
 			(at 166.37 59.69 0)
 			(effects
@@
 			)
 		)
-		(property "Footprint" "ScottoKeebs_Components:LED_SK6812MINI"
+		(property "Footprint" "Hackclub Footprints:MX_SK6812MINI-E_REV"
 			(at 128.27 59.69 0)
 			(effects
@@
 			)
 		)
-		(property "Footprint" "Seeed Studio XIAO Series Library:XIAO-RP2040-DIP"
+		(property "Footprint" "Hackclub Footprints:XIAO-RP2040-DIP"
 			(at 66.548 67.818 0)
 			(effects
@@
 			)
 		)
-		(property "Footprint" "ScottoKeebs_Components:LED_SK6812MINI"
+		(property "Footprint" "Hackclub Footprints:MX_SK6812MINI-E_REV"
 			(at 147.32 59.69 0)
 			(effects
